File: Hardware/01_Design/Input.kicad_sch (KiCad schematic)
At the start: 16 parts, among them J3 Conn_01x03, J4 Conn_01x03, SW2 SW_12x12mm_SMD, SW3 SW_12x12mm_SMD, SW4 SW_12x12mm_SMD, SW5 SW_12x12mm_SMD, U4 AM2302

Commit message: Placement component
Parts:
- added J3: Conn_01x05, Connector_PinHeader_2.54mm:PinHeader_1x05_P2.54mm_Vertical, symbol Measurement_Power_AC:Conn_01x05
- renumbered J3 to J5
Connections:
- new net T_CS: J3.4 (Pin_4)
- new net T_IRQ: J3.1 (Pin_1)
- new net T_MISO: J3.2 (Pin_2)
- new net T_MOSI: J3.3 (Pin_3)
- new net T_SCK: J3.5 (Pin_5)
Other:
- note added: "TFT TOUCH"
- moved on the sheet: J4, J5, R15, U4

Commit message: auto switch ver 1
Parts:
- removed SW2, SW3, SW4, SW5: SW_12x12mm_SMD, SW_12x12mm:SW_B3FS-4055P, symbol Measurement_Power_AC:SW_12x12mm_SMD
- added SW2, SW3, SW4, SW5: SW_6x6mm, Tactile_Switch_SMD:TE_FSM4JSMA, symbol Measurement_Power_AC:SW_6x6mm
- renumbered C25 to C21, C27 to C22, C26 to C23, C28 to C24, J5 to J3, J3 to J5, R13 to R12, R16 to R13, R17 to R15, R15 to R16, U4 to U3
Connections:
- net Button_1: now also SW2.1, SW2.2
- net Button_2: now also SW4.1, SW4.2
- net Button_3: now also SW3.1, SW3.2
- net Button_4: now also SW5.1, SW5.2
- net GND: now also SW2.3, SW2.4, SW3.3, SW3.4, SW4.3, SW4.4, SW5.3, SW5.4
- net LDR_A0 renamed LDR
