File: Hardware/01_Design/Output.kicad_sch (KiCad schematic)
At the start: 44 parts, among them J10 Conn_01x05, J11 Terminal, J5 Terminal, J6 Terminal, J7 Terminal, J8 Terminal, J9 Conn_01x08, K1 HF46F 12-HS1, K2 HF46F 12-HS1, K3 HF46F 12-HS1, K4 HF46F 12-HS1, Q1 MMBTA42, Q2 MMBTA42, Q3 MMBTA42, Q4 MMBTA42, U5 PC817X2NIPW, U6 PC817X2NIPW, U7 PC817X2NIPW, U8 PC817X2NIPW

Commit message: Placement component
Parts:
- removed J10: Conn_01x05, Connector_PinHeader_2.54mm:PinHeader_1x05_P2.54mm_Vertical, symbol Measurement_Power_AC:Conn_01x05
- removed J9: Conn_01x08, Connector_PinHeader_2.54mm:PinHeader_1x08_P2.54mm_Vertical, symbol Measurement_Power_AC:Conn_01x08
- added J10: Conn_01x08, Connector_PinHeader_2.54mm:PinHeader_1x08_P2.54mm_Vertical, symbol Measurement_Power_AC:Conn_01x08
- renumbered J5 to J6, J6 to J7, J7 to J8, J8 to J9
Connections:
- net +3V3: now also J10.1 (Pin_1), J10.8 (Pin_8)
- net GND: now also J10.7 (Pin_7)
- net TFT_CS: now also J10.6 (Pin_6)
- net TFT_DC: now also J10.4 (Pin_4)
- net TFT_MOSI: now also J10.3 (Pin_3)
- net TFT_RST: now also J10.5 (Pin_5)
- net TFT_SCK: now also J10.2 (Pin_2)
Other:
- note removed: "TFT TOUCH"
- moved on the sheet: D11, D12, D13, D14, J11, R30, R31, R32, R33, RV1

Commit message: auto switch ver 1
Parts:
- removed D11, D12, D13, D14: LED_0805, Measure_Power_AC:LED_0805, symbol Measurement_Power_AC:LED_0805
- removed J11, J6, J7, J8, J9: Terminal, charge_battery_footprint_lib:Terminal_2_P3.81mm, symbol charge_battery_sym_lib:Terminal_Block Plug-in_2P
- removed R30, R31, R32, R33: 1K/1%/1_10W, Measure_Power_AC:Res_0603, symbol Measurement_Power_AC:Res_1K_0603_1%
- added J10, J11, J6, J8, J9: Domino, Measure_Power_AC:Domino_2P, symbol charge_battery_sym_lib:Domino_2P
- RV1: footprint Measure_Power_AC:MOV07D471K -> Varistor:RV_Disc_D7mm_W3.4mm_P5mm
- renumbered D7 to D6, D9 to D7, D10 to D9, J10 to J7, K3 to K2, K2 to K3, Q3 to Q2, Q2 to Q3, R18 to R17, R24 to R18, R20 to R19, R26 to R20, R22 to R21, R28 to R22, R19 to R23, R25 to R24, R21 to R25, R27 to R26, R23 to R27, R29 to R28, U5 to U4, U7 to U5, U8 to U7
Connections:
- net AC1: now also J6.1
- net AC2: now also J10.1, J11.1, J6.2, J8.1, J9.1
- net LIGHT1_L: now reaches K3.4
- net LIGHT1_L: now also J10.2
- net FAN_L: now reaches K1.4
- net FAN_L: now also J8.2
- net LIGHT2_L: now reaches K2.4
- net LIGHT2_L: now also J9.2
- net DEHUM_L: now reaches K4.4
- net DEHUM_L: now also J11.2
Other:
- note removed: "LED"
