File: Hardware/01_Design/Power_Supply.kicad_sch (KiCad schematic)
At the start: 40 parts, among them J1 Jack_DC, U1 TPS54231DR, U2 AMS1117-3.3

Commit message: auto switch ver 1
Parts:
- removed C10, C13: 10uF/16V, Measure_Power_AC:Ceramic_Cap_0603, symbol DongKhoa:Ceramic_Cap_SMD_0603_10uF_16V
- removed C11, C12: 1uF/16V, Measure_Power_AC:Ceramic_Cap_0603, symbol DongKhoa:Ceramic_Cap_SMD_1uF_16V
- removed C6: 4.7nF/50V, charge_battery_footprint_lib:Ceramic_Cap_0603, symbol Measurement_Power_AC:Ceramic_Cap_SMD_4.7nF_50V
- removed C7: 39pF/50V, charge_battery_footprint_lib:Ceramic_Cap_0603, symbol Measurement_Power_AC:Ceramic_Cap_SMD_39pF_50V
- removed D4: LED_0805, Measure_Power_AC:LED_0805, symbol DongKhoa:LED_0805
- removed R2: 2.49K/1%/1_10W, Measure_Power_AC:Res_0603, symbol Measurement_Power_AC:Res_2.49K_0603_1%
- removed R5: 49.9K/1%/1_10W, Measure_Power_AC:Res_0603, symbol Measurement_Power_AC:Res_49.9K_0603_1%
- removed R8: 1K/1%/1_10W, Measure_Power_AC:Res_0603, symbol DongKhoa:Res_1K_0603_1%
- removed TP2: TestPoint, TestPoint:TestPoint_Pad_2.0x2.0mm, symbol DongKhoa:TestPoint
- removed U2: AMS1117-3.3, Package_TO_SOT_SMD:SOT-223-3_TabPin2, symbol DongKhoa:AMS1117-3.3
- added C4: 1nF/50V, Measure_Power_AC:Ceramic_Cap_0603, symbol Measurement_Power_AC:Ceramic_Cap_SMD_0603_1nF_50V
- added C5: 47pF/50V, Measure_Power_AC:Ceramic_Cap_0603, symbol Measurement_Power_AC:Ceramic_Cap_SMD_47pF_50V
- added FB1: 2A_120R, Measure_Power_AC:FB_0805, symbol DongKhoa:FerriteBead_2A_120R_Small
- added R7: 3K/1%/1_10W, Measure_Power_AC:Res_0603, symbol Measurement_Power_AC:Res_3K_0603_1%
- added R8: 220/1%/1_10W, charge_battery_footprint_lib:Res_0603, symbol charge_battery_sym_lib:Res_220R_0603_1%
- renumbered C2 to C1, C3 to C2, C9 to C3, C8 to C6, C1 to C7, C4 to C8, C5 to C9, D3 to D1, D5 to D3, D1 to D4, H3 to H2, H2 to H3, R3 to R2, R4 to R3, R7 to R4, R9 to R5, TP3 to TP2, TP4 to TP3
Connections:
- net +5V is gone; now on net +3V3: C8.2, C9.2, L1.1
- net +12V: now also FB1.1; no longer C1.2, C2.2, R1.2, U1.2 (VIN)
- net +3V3: now also R6.2
- net GND: now also C5.1, R8.1; no longer R6.1
- net VSENSE: now also R6.1, R7.2; no longer R6.2
- net at U1.6 (COMP): now also C4.2, C5.2
- net at R3.2: now also C4.1
- new net: R7.1, R8.2
- new net FB: C1.2, C2.2, FB1.2, R1.2, U1.2 (VIN)
Other:
- note removed: "LINEAR REGUALATOR 3V3 - AMS1117"
- moved on the sheet: D2, D3, H1, H2, H3, H4, R4, R5, TP1, TP2, TP3
