File: Hardware/01_Design/STM32.kicad_sch (KiCad schematic)
At the start: 19 parts, among them J2 Conn_01x04, SW1 EN, U3 STM32F103C8T6, Y1 8MHz_3225

Commit message: Placement component
Changed lines of the file:
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@@
 	(wire
 		(pts
-			(xy 49.53 100.33) (xy 53.34 100.33)
+			(xy 52.07 100.33) (xy 53.34 100.33)
 		)
 		(stroke
@@
 	)
 	(global_label "T_IRQ"
-		(shape output)
-		(at 49.53 100.33 180)
+		(shape input)
+		(at 52.07 100.33 180)
 		(fields_autoplaced yes)
 		(effects
@@
 		)
 		(property "Intersheetrefs" "${INTERSHEET_REFS}"
-			(at 41.4043 100.33 0)
+			(at 43.9443 100.33 0)
 			(hide yes)
 			(show_name no)

Commit message: auto switch ver 1
Parts:
- removed U3: STM32F103C8T6, Measure_Power_AC:STM32F103C8T6, symbol Measurement_Power_AC:STM32F103C8T6
- added U2: STM32F103C8T6, Lib:QFP50P900X900X160-48N, symbol Measurement_Power_AC:STM32F103C8T6
- Y1: Supply URL https://www.thegioiic.com/thach-anh-27-12mhz-3225-4-chan-smd -> https://www.thegioiic.com/thach-anh-8mhz-3225-4-chan-smd; Supply part number Thạch Anh 27.12MHz 3225 4 Chân SMD -> Thạch Anh 8MHz 3225 4 Chân SMD
- renumbered C19 to C10, C23 to C11, C20 to C12, C24 to C13, C17 to C14, C21 to C15, C18 to C17, C22 to C18, C14 to C19, C15 to C20, D6 to D5, R12 to R11, R11 to R9
Connections:
- net +3V3: now also U2.24 (VDD_1), U2.36 (VDD_2), U2.48 (VDD_3), U2.9 (VDDA)
- net BOOT0: now also U2.44 (BOOT0)
- net Button_1: now also U2.13 (PA3)
- net Button_2: now also U2.20 (PB2)
- net Button_3: now also U2.31 (PA10)
- net Button_4: now also U2.32 (PA11-CAN_RX)
- net DEHUMIDIFER: now also U2.33 (PA12-CAN_TX)
- net DHT22: now also U2.45 (PB8)
- net FAN: now also U2.40 (PB4)
- net GND: now also U2.23 (VSS_1), U2.35 (VSS_2), U2.47 (VSS_3), U2.8 (VSSA)
- net LED_STATUS: now also U2.2 (PC13)
- net LIGHT_1: now also U2.38 (PA15)
- net LIGHT_2: now also U2.42 (PB6)
- net NRST: now also U2.7 (NRST)
- net OSC_IN: now also U2.5 (PD0-OSC_IN-RCC_OSC_IN)
- net OSC_OUT: now also U2.6 (PD1-OSC_OUT-RCC_OSC_OUT)
- net PIR: now also U2.30 (PA9)
- net SWCLK: now also U2.37 (PA14-SYS_JTCK-SWCLK)
- net SWDIO: now also U2.34 (PA13-SYS_JTMS-SWDIO)
- net TFT_CS: now also U2.14 (PA4)
- net TFT_DC: now also U2.18 (PB0)
- net TFT_MOSI: now also U2.17 (PA7)
- net TFT_RST: now also U2.19 (PB1)
- net TFT_SCK: now also U2.15 (PA5)
- net T_CS: now also U2.25 (PB12)
- net T_IRQ: now also U2.22 (PB11)
- net T_MISO: now also U2.27 (PB14)
- net T_MOSI: now also U2.28 (PB15)
- net T_SCK: now also U2.26 (PB13)
- new net LDR: U2.21 (PB10)
- no-connect marks 7 -> 12
