File: Hardware/01_Design/Smart_Switch.kicad_pcb (KiCad board)
At the start: 2 copper layers, 100 x 67.2 mm, 119 parts, among them J1 Jack_DC, J10 Conn_01x08, J11 Terminal, J2 Conn_01x04, J3 Conn_01x05, J4 Conn_01x03, J5 Conn_01x03, J6 Terminal, J7 Terminal, J8 Terminal, J9 Terminal, K1 HF46F 12-HS1, K2 HF46F 12-HS1, K3 HF46F 12-HS1, K4 HF46F 12-HS1, Q1 MMBTA42, Q2 MMBTA42, Q3 MMBTA42, Q4 MMBTA42, SW1 EN, SW2 SW_12x12mm_SMD, SW3 SW_12x12mm_SMD, SW4 SW_12x12mm_SMD, SW5 SW_12x12mm_SMD, U1 TPS54231DR, U2 AMS1117-3.3, U3 STM32F103C8T6, U4 AM2302, U5 PC817X2NIPW, U6 PC817X2NIPW, U7 PC817X2NIPW, U8 PC817X2NIPW, Y1 8MHz_3225

Commit message: Update
Parts:
- added J11: Conn_01x02, Connector_PinHeader_2.54mm:PinHeader_1x02_P2.54mm_Horizontal, F.Cu at (1.79, 30.4)
- added J6: Conn_01x02, Connector_PinHeader_2.54mm:PinHeader_1x02_P2.54mm_Horizontal, F.Cu at (1.79, 1.79)
- added J7: Conn_01x02, Connector_PinHeader_2.54mm:PinHeader_1x02_P2.54mm_Horizontal, F.Cu at (1.79, 8.94)
- added J8: Conn_01x02, Connector_PinHeader_2.54mm:PinHeader_1x02_P2.54mm_Horizontal, F.Cu at (1.79, 16.1)
- added J9: Conn_01x02, Connector_PinHeader_2.54mm:PinHeader_1x02_P2.54mm_Horizontal, F.Cu at (1.79, 23.2)
Connections:
- K1 pad 4: Net-(J6-Pad2) -> Net-(J6-Pin_2)
- K2 pad 4: Net-(J7-Pad2) -> Net-(J7-Pin_2)
- K3 pad 4: Net-(J8-Pad2) -> Net-(J8-Pin_2)
- K4 pad 4: Net-(J9-Pad2) -> Net-(J9-Pin_2)

Commit message: auto switch ver 1
Parts:
- removed the C10 at (165.9, 79.8)
- removed the C11 at (163.6, 79.8)
- removed the C12 at (163.4, 83.6)
- removed the C13 at (165.7, 83.6)
- removed the C6 at (169.5, 95.7)
- removed the C7 at (167.6, 95.7)
- removed D11, D12, D13, D14: LED_0805, Measure_Power_AC:LED_0805
- removed the D4 at (146.3, 229.5)
- removed the J11 at (1.79, 30.4)
- removed the J11 at (235.6, 79.4)
- removed the J6 at (1.79, 1.79)
- removed the J6 at (243.0, 90.9)
- removed the J7 at (1.79, 8.94)
- removed the J7 at (243.2, 103.6)
- removed the J8 at (1.79, 16.1)
- removed the J8 at (243.2, 117.6)
- removed the J9 at (1.79, 23.2)
- removed the J9 at (243.2, 130.3)
- removed the R2 at (166.1, 93.8)
- removed R30, R31, R32, R33: 1K/1%/1_10W, Measure_Power_AC:Res_0603
- removed the R5 at (169.9, 91.1)
- removed the TP2 at (164.8, 218.6)
- removed the U3 at (184.2, 92.7)
- added C4: 1nF/50V, Measure_Power_AC:Ceramic_Cap_0603, F.Cu at (170.0, 98.3)
- added C5: 47pF/50V, Measure_Power_AC:Ceramic_Cap_0603, F.Cu at (168.0, 98.3)
- added FB1: 2A_120R, Measure_Power_AC:FB_0805, F.Cu at (151.8, 93.6)
- added G***: LOGO, logo:BKU_name, F.Cu at (216.4, 78.5)
- added J10: Domino, Measure_Power_AC:Domino_2P, F.Cu at (242.4, 105.9)
- added J11: Domino, Measure_Power_AC:Domino_2P, F.Cu at (242.4, 132.7)
- added J6: Domino, Measure_Power_AC:Domino_2P, F.Cu at (226.6, 138.9)
- added J8: Domino, Measure_Power_AC:Domino_2P, F.Cu at (242.4, 93.2)
- added J9: Domino, Measure_Power_AC:Domino_2P, F.Cu at (242.4, 119.2)
- added R7: 3K/1%/1_10W, Measure_Power_AC:Res_0603, F.Cu at (171.4, 85.9)
- C16, Q1, Q4, R14: moved to B.Cu
- C21: renamed from C25; moved to B.Cu
- C22: renamed from C27; moved to B.Cu
- C23: renamed from C26; moved to B.Cu
- C24: renamed from C28; moved to B.Cu
- Q2: renamed from Q3; moved to B.Cu
- Q3: renamed from Q2; moved to B.Cu
- R11: renamed from R12; moved to B.Cu
- R12: renamed from R13; moved to B.Cu
- R13: renamed from R16; moved to B.Cu
- R15: renamed from R17; moved to B.Cu
- R16: renamed from R15; moved to B.Cu
- R17: renamed from R18; moved to B.Cu
- R18: renamed from R24; moved to B.Cu
- R19: renamed from R20; moved to B.Cu
- R20: renamed from R26; moved to B.Cu
- R21: renamed from R22; moved to B.Cu
- R22: renamed from R28; moved to B.Cu
- R23: renamed from R19; moved to B.Cu
- R24: renamed from R25; moved to B.Cu
- R25: renamed from R21; moved to B.Cu
- R26: renamed from R27; moved to B.Cu
- R27: renamed from R23; moved to B.Cu
- R28: renamed from R29; moved to B.Cu
- R4: renamed from R7; moved to B.Cu
- R5: renamed from R9; moved to B.Cu
- R6: moved to F.Cu
- R8: value 1K/1%/1_10W -> 220/1%/1_10W; footprint Measure_Power_AC:Res_0603 -> charge_battery_footprint_lib:Res_0603
- R9: renamed from R11; moved to B.Cu
- RV1: footprint Measure_Power_AC:MOV07D471K -> Varistor:RV_Disc_D7mm_W3.4mm_P5mm
- SW2, SW3, SW4, SW5: value SW_12x12mm_SMD -> SW_6x6mm; footprint SW_12x12mm:SW_B3FS-4055P -> Tactile_Switch_SMD:TE_FSM4JSMA
- U2: value AMS1117-3.3 -> STM32F103C8T6; footprint Package_TO_SOT_SMD:SOT-223-3_TabPin2 -> Lib:QFP50P900X900X160-48N
- moved R4 151.3 mm to (159.4, 78.4), turned to -90 degrees
- moved R8 149.1 mm to (173.4, 84.6), turned to -90 degrees
- moved D2 146.5 mm to (163.8, 80.9), turned to -90 degrees
- moved TP3 137.9 mm to (188.6, 90.9)
- moved TP1 133.5 mm to (159.6, 81.1)
- moved C14 127.7 mm to (176.7, 102.9), turned to 180 degrees
- moved C17 127.1 mm to (170.0, 101.9), turned to 90 degrees
- moved R10 126.8 mm to (171.3, 100.6), turned to -90 degrees
- moved R11 124.3 mm to (162.0, 104.5), turned to 180 degrees
- moved D5 121.8 mm to (160.7, 103.8)
- moved Y1 121.1 mm to (160.7, 109.2), turned to 180 degrees
- moved C18 120.2 mm to (168.0, 101.9), turned to 90 degrees
- moved C15 120.1 mm to (176.7, 104.8), turned to 180 degrees
- moved C13 117.6 mm to (177.9, 115.6), turned to 90 degrees
- moved D3 117.1 mm to (191.3, 124.3), turned to 90 degrees
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- renumbered C2 to C1, C19 to C10, C23 to C11, C20 to C12, C24 to C13, C17 to C14, C21 to C15, C18 to C17, C22 to C18, C14 to C19, C3 to C2, C15 to C20, C9 to C3, C8 to C6, C1 to C7, C4 to C8, C5 to C9, D3 to D1, D5 to D3, D1 to D4, D6 to D5, D7 to D6, D9 to D7, D10 to D9, H3 to H2, H2 to H3, J5 to J3, J3 to J5, J10 to J7, K3 to K2, K2 to K3, R3 to R2, R4 to R3, TP3 to TP2, TP4 to TP3, U4 to U3, U5 to U4, U7 to U5, U8 to U7
Connections:
- C1 pad 2: +12V -> /Power_Supply/FB
- C2 pad 2: +12V -> /Power_Supply/FB
- C8 pad 2: +5V -> +3V3
- C9 pad 2: +5V -> +3V3
- J4 pad 3: LDR_A0 -> LDR
- K1 pad 4: Net-(J6-Pin_2) -> /Output/FAN_L
- K2 pad 4: Net-(J8-Pin_2) -> /Output/LIGHT2_L
- K3 pad 4: Net-(J7-Pin_2) -> /Output/LIGHT1_L
- K4 pad 4: Net-(J9-Pin_2) -> /Output/DEHUM_L
- L1 pad 1: +5V -> +3V3
- R1 pad 2: +12V -> /Power_Supply/FB
- R6 pad 1: GND -> /Power_Supply/VSENSE
- R6 pad 2: /Power_Supply/VSENSE -> +3V3
- R8 pad 1: Net-(D4-K) (its old number) -> GND
- R8 pad 2: GND -> Net-(R7-Pad1)
- SW3 pad 1: Button_2 -> Button_3
- SW3 pad 2: Button_2 -> Button_3
- SW4 pad 1: Button_3 -> Button_2
- SW4 pad 2: Button_3 -> Button_2
- U1 pad 2: +12V -> /Power_Supply/FB
- U2 pad 1: GND -> unconnected-(U2B-VBAT-Pad1)
- U2 pad 2: +3V3 -> /STM32/LED_STATUS
- U2 pad 3: +5V -> unconnected-(U2A-PC14-OSC32_IN-Pad3)
Routing:
- net GND: track 0.00 -> 433.3 mm, vias 0 -> 104
- net +3V3: track 0.00 -> 329.0 mm, vias 0 -> 6
- net +12V: track 0.00 -> 143.4 mm, vias 0 -> 8
- net Button_4: track 0.00 -> 58.1 mm, vias 0 -> 2
- net Button_3: track 0.00 -> 51.0 mm, vias 0 -> 1
- net Button_2: track 0.00 -> 47.7 mm, vias 0 -> 1
- net DEHUMIDIFER: track 0.00 -> 39.5 mm
- net PIR: track 0.00 -> 35.3 mm, vias 0 -> 1
- net FAN: track 0.00 -> 35.0 mm
- net DHT22: track 0.00 -> 35.0 mm, vias 0 -> 1
- net Button_1: track 0.00 -> 34.7 mm, vias 0 -> 2
- net /Power_Supply/VSENSE: track 0.00 -> 34.5 mm, vias 0 -> 2
- net LIGHT_2: track 0.00 -> 31.8 mm, vias 0 -> 2
- net LDR: track 0.00 -> 30.3 mm, vias 0 -> 1
- net LIGHT_1: track 0.00 -> 28.5 mm, vias 0 -> 2
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- added copper zone on B.Cu, net +12V
- added copper zone on F.Cu, net +12V
- added copper zone on F.Cu, net +3V3
- added copper zone on B.Cu, net /Output/AC1
- added copper zone on F.Cu, net /Output/AC2
- added copper zone on B.Cu, net /Output/DEHUM_L
- added copper zone on B.Cu, net /Output/FAN_L
- added copper zone on B.Cu, net /Output/LIGHT1_L
- added copper zone on B.Cu, net /Output/LIGHT2_L
- added copper zone on F.Cu, net /Power_Supply/FB
- added copper zone on B.Cu, net /Power_Supply/Fuse
- added copper zone on F.Cu, net /Power_Supply/Fuse
- added copper zone on B.Cu, net GND
- added copper zone on F.Cu, net GND
- added copper zone on F.Cu, net Net-(C4-Pad1)
- added copper zone on B.Cu, net Net-(D4-K)
- added copper zone on F.Cu, net Net-(D4-K)
- added copper zone on F.Cu, net Net-(U1-COMP)
Other:
- board size 100 x 67.2 mm -> 100 x 70 mm
- board text added: "12V"
- board text added: "220VAC"
- board text added: "3V3"
- board text added: "AUTO_SWITCH_VER 1"
- board text added: "CS"
- board text added: "DC"
- board text added: "DEHUMIDIFER"
- board text added: "DHT22"
- board text added: "FAN"
- board text added: "GND"
- board text added: "IRQ"
- board text added: "LDR"
- board text added: "LED TEST"
- board text added: "LIGHT"
- board text added: "LIGHT 1"
- board text added: "LIGHT 2"
- board text added: "LOAD"
- board text added: "MISO"
- board text added: "MODE"
- board text added: "MOSI"
- board text added: "PIR"
- board text added: "RESET"
- board text added: "RST"
- board text added: "SCK"
- board text added: "SWCLK"
- board text added: "SWDIO"
- board text added: "TOUCH"
- board text added: "Vu Dinh Khanh Linh Do Ngoc Tri Cuong Huynh Tan Phuc"
